File: EAGLE BoosterPack v2/Tricorder-BoosterPack.brd (EAGLE design)
At the start: 63.5 x 34.3 mm, 35 parts, among them U1 MAG3110, U2 LMT70LMT70, U3 HDC1000, U4 OPT3001, U5 LMP91000

Commit message: v2 PCB Layout
Revamped the PCB layout to make room for a PGA900 and Honeywell
Pressure Sensor
Parts:
- moved R7 7.79 mm to (38.2, 8.55)
- moved R3 5.08 mm to (45.9, 34.0)
- moved R4 5.08 mm to (47.4, 34.0)
- moved R5 5.08 mm to (48.9, 34.0)
- moved R8 5.08 mm to (22.5, 33.2)
- moved U$2 5.08 mm to (54.6, 35.8)
- moved C4 5.08 mm to (21.5, 19.5)
- moved C1 5.08 mm to (18.2, 23.8)
- moved C7 5.08 mm to (28.1, 20.8)
- moved SV1 5.08 mm to (37.0, 29.6)
- moved U5 5.08 mm to (30.2, 24.7)
- moved A1 5.08 mm to (9.79, 21.5)
- moved C3 5.08 mm to (22.3, 15.9)
- moved C6 5.08 mm to (25.1, 21.2)
- moved JP1 5.08 mm to (22.3, 28.1)
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Routing:
- net GND: track 61.7 -> 65.3 mm
- net BTN0: track 22.0 -> 25.1 mm
- net BTN1: track 33.5 -> 34.2 mm
Other:
- board size 63.5 x 34.3 mm -> 63.6 x 39.2 mm
