File: EAGLE BoosterPack v2/Tricorder-BoosterPack.sch (EAGLE design)
At the start: 34 parts, among them U1 MAG3110, U2 LMT70LMT70, U3 HDC1000, U4 OPT3001, U5 LMP91000

Commit message: v2 PCB Layout
Revamped the PCB layout to make room for a PGA900 and Honeywell
Pressure Sensor
Other:
- moved on the sheet: C2, JP1, R11, R9, U4, U5
