File: EAGLE BoosterPack rev2/Tricorder-BoosterPack.sch (EAGLE design)
At the start: 39 parts, among them U1 MAG3110, U2 LMT70LMT70, U3 HDC1000, U4 OPT3001, U5 LMP91000, U6 PGA900, U7 MICROSD

Commit message: Revised BOM
Parts:
- U5: DIGIKEY (none) -> LMP91000
Connections:
- net GND: now also U6.CSN
Other:
- moved on the sheet: C9, U5
Changed lines of the file:
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@@
 <part name="C6" library="adafruit" deviceset="C-US" device="C0603" value="1u"/>
 <part name="C7" library="adafruit" deviceset="C-US" device="C0603" value="100n"/>
-<part name="U5" library="LMP91000" deviceset="LMP91000" device=""/>
+<part name="U5" library="LMP91000" deviceset="LMP91000" device="">
+<attribute name="DIGIKEY" value="LMP91000"/>
+</part>
 <part name="GND20" library="supply1" deviceset="GND" device=""/>
 <part name="GND21" library="supply1" deviceset="GND" device=""/>
@@
 <part name="GND19" library="supply1" deviceset="GND" device=""/>
 <part name="GND15" library="supply1" deviceset="GND" device=""/>
+<part name="GND30" library="supply1" deviceset="GND" device=""/>
 </parts>
 <sheets>
@@
 <instance part="C6" gate="G$1" x="93.98" y="17.78"/>
 <instance part="C7" gate="G$1" x="83.82" y="17.78"/>
-<instance part="U5" gate="G$1" x="76.2" y="78.74"/>
+<instance part="U5" gate="G$1" x="73.66" y="78.74">
+<attribute name="DIGIKEY" x="68.58" y="45.72" size="1.778" layer="96"/>
+</instance>
 <instance part="GND20" gate="1" x="111.76" y="43.18"/>
 <instance part="GND21" gate="1" x="104.14" y="43.18"/>
@@
 <instance part="R11" gate="G$1" x="193.04" y="78.74"/>
 <instance part="JP2" gate="A" x="119.38" y="15.24"/>
-<instance part="C9" gate="G$1" x="50.8" y="53.34"/>
+<instance part="C9" gate="G$1" x="48.26" y="55.88"/>
 <instance part="GND6" gate="1" x="45.72" y="83.82" rot="R90"/>
 <instance part="U7" gate="G$1" x="218.44" y="170.18" rot="R90"/>
@@
 <instance part="GND19" gate="1" x="101.6" y="5.08"/>
 <instance part="GND15" gate="1" x="22.86" y="5.08"/>
+<instance part="GND30" gate="1" x="111.76" y="76.2"/>
 </instances>
 <busses>
@@
 <segment>
 <pinref part="U5" gate="G$1" pin="VDD"/>
-<wire x1="93.98" y1="81.28" x2="99.06" y2="81.28" width="0.1524" layer="91"/>
+<wire x1="91.44" y1="81.28" x2="99.06" y2="81.28" width="0.1524" layer="91"/>
 <label x="99.06" y="81.28" size="1.778" layer="95"/>
 </segment>
@@
 <pinref part="U5" gate="G$1" pin="DGND"/>
 <pinref part="GND20" gate="1" pin="GND"/>
-<wire x1="93.98" y1="60.96" x2="111.76" y2="60.96" width="0.1524" layer="91"/>
+<wire x1="91.44" y1="60.96" x2="111.76" y2="60.96" width="0.1524" layer="91"/>
 <wire x1="111.76" y1="60.96" x2="111.76" y2="45.72" width="0.1524" layer="91"/>
 </segment>
@@
 <pinref part="U5" gate="G$1" pin="AGND"/>
 <pinref part="GND21" gate="1" pin="GND"/>
-<wire x1="93.98" y1="55.88" x2="104.14" y2="55.88" width="0.1524" layer="91"/>
+<wire x1="91.44" y1="55.88" x2="104.14" y2="55.88" width="0.1524" layer="91"/>
 <wire x1="104.14" y1="55.88" x2="104.14" y2="45.72" width="0.1524" layer="91"/>
 </segment>
@@
 <wire x1="33.02" y1="17.78" x2="22.86" y2="17.78" width="0.1524" layer="91"/>
 <wire x1="22.86" y1="17.78" x2="22.86" y2="7.62" width="0.1524" layer="91"/>
+</segment>
+<segment>
+<pinref part="U6" gate="A" pin="CSN"/>
+<pinref part="GND30" gate="1" pin="GND"/>
+<wire x1="119.38" y1="81.28" x2="111.76" y2="81.28" width="0.1524" layer="91"/>
+<wire x1="111.76" y1="81.28" x2="111.76" y2="78.74" width="0.1524" layer="91"/>
 </segment>
 </net>
@@
 <segment>
 <pinref part="U5" gate="G$1" pin="SCL"/>
-<wire x1="93.98" y1="76.2" x2="99.06" y2="76.2" width="0.1524" layer="91"/>
+<wire x1="91.44" y1="76.2" x2="99.06" y2="76.2" width="0.1524" layer="91"/>
 <label x="99.06" y="76.2" size="1.778" layer="95"/>
 </segment>
@@
 <segment>
 <pinref part="U5" gate="G$1" pin="SDA"/>
-<wire x1="93.98" y1="71.12" x2="99.06" y2="71.12" width="0.1524" layer="91"/>
+<wire x1="91.44" y1="71.12" x2="99.06" y2="71.12" width="0.1524" layer="91"/>
 <label x="99.06" y="71.12" size="1.778" layer="95"/>
 </segment>
@@
 <segment>
 <pinref part="U5" gate="G$1" pin="MENB"/>
-<wire x1="93.98" y1="66.04" x2="99.06" y2="66.04" width="0.1524" layer="91"/>
+<wire x1="91.44" y1="66.04" x2="99.06" y2="66.04" width="0.1524" layer="91"/>
 <label x="99.06" y="66.04" size="1.778" layer="95"/>
 </segment>
@@
 <segment>
 <pinref part="U5" gate="G$1" pin="VOUT"/>
-<wire x1="93.98" y1="50.8" x2="96.52" y2="50.8" width="0.1524" layer="91"/>
+<wire x1="91.44" y1="50.8" x2="96.52" y2="50.8" width="0.1524" layer="91"/>
 <label x="96.52" y="50.8" size="1.778" layer="95" xref="yes"/>
 </segment>
@@
 <segment>
 <pinref part="U5" gate="G$1" pin="CE"/>
-<wire x1="58.42" y1="86.36" x2="53.34" y2="86.36" width="0.1524" layer="91"/>
+<wire x1="55.88" y1="86.36" x2="53.34" y2="86.36" width="0.1524" layer="91"/>
 <label x="50.8" y="86.36" size="1.778" layer="95"/>
 </segment>
@@
 <segment>
 <pinref part="U5" gate="G$1" pin="RE"/>
-<wire x1="58.42" y1="81.28" x2="53.34" y2="81.28" width="0.1524" layer="91"/>
+<wire x1="55.88" y1="81.28" x2="53.34" y2="81.28" width="0.1524" layer="91"/>
 <label x="50.8" y="81.28" size="1.778" layer="95"/>
 </segment>
@@
 <segment>
 <pinref part="U5" gate="G$1" pin="WE"/>
-<wire x1="58.42" y1="76.2" x2="53.34" y2="76.2" width="0.1524" layer="91"/>
+<wire x1="55.88" y1="76.2" x2="53.34" y2="76.2" width="0.1524" layer="91"/>
 <label x="50.8" y="76.2" size="1.778" layer="95"/>
 </segment>
@@
 <segment>
 <pinref part="C9" gate="G$1" pin="1"/>
-<wire x1="50.8" y1="55.88" x2="50.8" y2="66.04" width="0.1524" layer="91"/>
+<wire x1="48.26" y1="58.42" x2="50.8" y2="66.04" width="0.1524" layer="91"/>
 <pinref part="U5" gate="G$1" pin="C1"/>
-<wire x1="50.8" y1="66.04" x2="58.42" y2="66.04" width="0.1524" layer="91"/>
-</segment>
-</net>
-<net name="N$13" class="0">
+<wire x1="50.8" y1="66.04" x2="55.88" y2="66.04" width="0.1524" layer="91"/>
+</segment>
+</net>
+<net name="N$11" class="0">
 <segment>
 <pinref part="U5" gate="G$1" pin="C2"/>
-<wire x1="58.42" y1="60.96" x2="55.88" y2="60.96" width="0.1524" layer="91"/>
-<wire x1="55.88" y1="60.96" x2="55.88" y2="45.72" width="0.1524" layer="91"/>
+<wire x1="55.88" y1="60.96" x2="53.34" y2="60.96" width="0.1524" layer="91"/>
+<wire x1="53.34" y1="60.96" x2="53.34" y2="45.72" width="0.1524" layer="91"/>
 <pinref part="C9" gate="G$1" pin="2"/>
-<wire x1="55.88" y1="45.72" x2="50.8" y2="45.72" width="0.1524" layer="91"/>
-<wire x1="50.8" y1="45.72" x2="50.8" y2="48.26" width="0.1524" layer="91"/>
-</segment>
-</net>
+<wire x1="53.34" y1="45.72" x2="50.8" y2="45.72" width="0.1524" layer="91"/>
+<wire x1="50.8" y1="45.72" x2="48.26" y2="50.8" width="0.1524" layer="91"/>
+</segment>
+</net>
